File: pcb/pmw3610/pmw3610.kicad_sch (KiCad schematic)
At the start: 18 parts, among them J2 Conn_01x06_Female, J3 Conn_01x06_Female, U1 TCR2EF19, U2 PMW3610

Commit message: updated to add alternate parts for the LDO for the vik pmw3610 module
Parts:
- U1: LCSC-alternate-1 (none) -> C2862411; LCSC-alternate-2 (none) -> C2869109
Changed lines of the file:
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@@
+      (effects (font (size 1.27 1.27)) hide)
+    )
+    (property "LCSC-alternate-1" "C2862411" (at 64.008 54.356 0)
+      (effects (font (size 1.27 1.27)) hide)
+    )
+    (property "LCSC-alternate-2" "C2869109" (at 64.008 54.356 0)
       (effects (font (size 1.27 1.27)) hide)
     )
